File: hardware/esp32-iot-uno/esp32-iot-uno-hw.sch (KiCad schematic (older format))
At the start: 91 parts, among them CON1 BARREL_JACK, P1 GPIO, P2 GPIO, P3 ADC, P4 GPIO, P5 OLED, Q1 S8050_NPN_BEC, Q2 S8050_NPN_BEC, SW1 SW_EN, SW2 SW_IO18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

Commit message: Working on BOM.
Parts:
- U3: value CP2102 -> CP2109
Changed lines of the file:
@@
-$EndComp
-$Comp
-L usb_mini_b:usb_mini_b U1
-U 1 1 5888B18B
-P 1300 5400
-F 0 "U1" H 1250 6097 60  0000 C CNN
-F 1 "usb_mini_b" H 1250 5991 60  0000 C CNN
-F 2 "Connectors:USB_Micro-B" H 300 5850 60  0001 C CNN
-F 3 "" H 300 5850 60  0000 C CNN
-	1    1300 5400
-	1    0    0    -1
 $EndComp
 $Comp
@@
 	1    0    0    -1
 $EndComp
-NoConn ~ 750  5100
-NoConn ~ 750  5200
-NoConn ~ 750  5300
 $Comp
 L esp32-iot-uno-hw-rescue:BARREL_JACK CON1
@@
 Text GLabel 6200 3800 2    60   Input ~ 0
 CLK/GPIO6
-$Comp
-L CP2102:CP2102 U3
-U 1 1 5893B91A
-P 2550 7100
-F 0 "U3" H 2550 7200 50  0000 C CNN
-F 1 "CP2102" H 2550 7100 50  0000 C CNN
-F 2 "Housings_DFN_QFN:QFN-28-1EP_5x5mm_Pitch0.5mm" H 2550 7100 60  0001 C CNN
-F 3 "" H 2550 7100 60  0001 C CNN
-	1    2550 7100
-	1    0    0    -1
-$EndComp
 Text GLabel 1100 6750 0    60   Input ~ 0
 D-
@@
 F 3 "" H 3250 6200 50  0000 C CNN
 	1    3250 6200
-	1    0    0    -1
-$EndComp
-$Comp
-L esp32-iot-uno-hw-rescue:C_Small C20
-U 1 1 5893EAD9
-P 3550 6200
-F 0 "C20" H 3642 6246 50  0000 L CNN
-F 1 "10uF" H 3642 6155 50  0000 L CNN
-F 2 "footprint:C_0603" H 3550 6200 50  0001 C CNN
-F 3 "" H 3550 6200 50  0000 C CNN
-	1    3550 6200
 	1    0    0    -1
 $EndComp
@@
 Wire Wire Line
 	12925 9450 12925 9650
-Wire Wire Line
-	750  5000 700  5000
 Connection ~ 1250 5550
 Wire Wire Line
@@
 Connection ~ 3000 6050
 Wire Wire Line
-	3550 6050 3550 6100
-Connection ~ 3250 6050
-Wire Wire Line
 	3250 6300 3250 6350
-Wire Wire Line
-	3250 6350 3550 6350
-Connection ~ 3550 6350
 Wire Wire Line
 	2900 5300 2900 5800
@@
 Wire Wire Line
 	3900 6350 3900 6400
-Wire Wire Line
-	3550 6300 3550 6350
 Wire Wire Line
 	12750 1400 12750 1425
@@
 	3000 6050 3000 6150
 Wire Wire Line
+	3100 6050 3250 6050
+Wire Wire Line
+	2900 5800 2900 6150
+Wire Wire Line
+	2500 5800 2900 5800
+Wire Wire Line
+	2300 6100 2500 6100
+Wire Wire Line
+	5400 6800 5550 6800
+Wire Wire Line
+	5400 7500 5550 7500
+Wire Wire Line
+	8100 2400 8100 2450
+Wire Wire Line
+	1350 3650 1350 3750
+Wire Wire Line
+	1950 3650 1950 3750
+Wire Wire Line
+	10400 1550 10400 1650
+Wire Wire Line
+	13100 6550 13250 6550
+Wire Wire Line
+	8100 2700 8100 2750
+Wire Wire Line
+	12750 1425 12750 1500
+Wire Wire Line
+	12750 1825 12750 1900
+Wire Wire Line
+	13100 1425 13250 1425
+Wire Wire Line
+	12750 3975 12750 4075
+Wire Wire Line
+	12750 2950 12750 3050
+Wire Wire Line
+	12750 2575 12750 2625
+Wire Wire Line
+	12750 3650 12750 3675
+Wire Wire Line
+	13025 2575 13250 2575
+Wire Wire Line
+	13050 3650 13250 3650
+Wire Wire Line
+	14650 1400 14650 1525
+Wire Wire Line
+	14850 1400 15100 1400
+Wire Wire Line
+	14650 1825 14650 1900
+Wire Wire Line
+	14650 2900 14650 3000
+Wire Wire Line
+	14650 2575 14650 2625
+Wire Wire Line
+	14900 2575 15100 2575
+Wire Wire Line
+	14650 3675 14650 3725
+Wire Wire Line
+	14650 4025 14650 4100
+Wire Wire Line
+	14900 3675 15175 3675
+Wire Wire Line
+	8250 6000 8600 6000
+Wire Wire Line
+	9850 6000 10200 6000
+Wire Wire Line
+	10200 6000 10350 6000
+Wire Wire Line
+	8150 6000 8250 6000
+Wire Wire Line
+	10550 5700 10900 5700
+Wire Wire Line
+	10900 6000 10900 6300
+Wire Wire Line
+	10900 6000 11050 6000
+Wire Wire Line
+	10900 5700 11450 5700
+Wire Wire Line
+	7850 6000 7850 6250
+Wire Wire Line
+	6150 9950 6150 10050
+Wire Wire Line
+	7550 9950 8000 9950
+Wire Wire Line
+	750  5000 700  5000
+NoConn ~ 750  5300
+NoConn ~ 750  5200
+NoConn ~ 750  5100
+$Comp
+L usb_mini_b:usb_mini_b U1
+U 1 1 5888B18B
+P 1300 5400
+F 0 "U1" H 1250 6097 60  0000 C CNN
+F 1 "usb_mini_b" H 1250 5991 60  0000 C CNN
+F 2 "Connectors:USB_Micro-B" H 300 5850 60  0001 C CNN
+F 3 "" H 300 5850 60  0000 C CNN
+	1    1300 5400
+	1    0    0    -1
+$EndComp
+Connection ~ 3550 6350
+Wire Wire Line
+	3550 6350 3900 6350
+Wire Wire Line
+	3250 6350 3550 6350
+Connection ~ 3250 6050
+Wire Wire Line
 	3250 6050 3550 6050
 Wire Wire Line
-	3550 6350 3900 6350
-Wire Wire Line
-	3100 6050 3250 6050
-Wire Wire Line
-	2900 5800 2900 6150
-Wire Wire Line
-	2500 5800 2900 5800
-Wire Wire Line
-	2300 6100 2500 6100
-Wire Wire Line
-	5400 6800 5550 6800
-Wire Wire Line
-	5400 7500 5550 7500
-Wire Wire Line
-	8100 2400 8100 2450
-Wire Wire Line
-	1350 3650 1350 3750
-Wire Wire Line
-	1950 3650 1950 3750
-Wire Wire Line
-	10400 1550 10400 1650
-Wire Wire Line
-	13100 6550 13250 6550
-Wire Wire Line
-	8100 2700 8100 2750
-Wire Wire Line
-	12750 1425 12750 1500
-Wire Wire Line
-	12750 1825 12750 1900
-Wire Wire Line
-	13100 1425 13250 1425
-Wire Wire Line
-	12750 3975 12750 4075
-Wire Wire Line
-	12750 2950 12750 3050
-Wire Wire Line
-	12750 2575 12750 2625
-Wire Wire Line
-	12750 3650 12750 3675
-Wire Wire Line
-	13025 2575 13250 2575
-Wire Wire Line
-	13050 3650 13250 3650
-Wire Wire Line
-	14650 1400 14650 1525
-Wire Wire Line
-	14850 1400 15100 1400
-Wire Wire Line
-	14650 1825 14650 1900
-Wire Wire Line
-	14650 2900 14650 3000
-Wire Wire Line
-	14650 2575 14650 2625
-Wire Wire Line
-	14900 2575 15100 2575
-Wire Wire Line
-	14650 3675 14650 3725
-Wire Wire Line
-	14650 4025 14650 4100
-Wire Wire Line
-	14900 3675 15175 3675
-Wire Wire Line
-	8250 6000 8600 6000
-Wire Wire Line
-	9850 6000 10200 6000
-Wire Wire Line
-	10200 6000 10350 6000
-Wire Wire Line
-	8150 6000 8250 6000
-Wire Wire Line
-	10550 5700 10900 5700
-Wire Wire Line
-	10900 6000 10900 6300
-Wire Wire Line
-	10900 6000 11050 6000
-Wire Wire Line
-	10900 5700 11450 5700
-Wire Wire Line
-	7850 6000 7850 6250
-Wire Wire Line
-	6150 9950 6150 10050
-Wire Wire Line
-	7550 9950 8000 9950
+	3550 6300 3550 6350
+Wire Wire Line
+	3550 6050 3550 6100
+$Comp
+L esp32-iot-uno-hw-rescue:C_Small C20
+U 1 1 5893EAD9
+P 3550 6200
+F 0 "C20" H 3642 6246 50  0000 L CNN
+F 1 "10uF" H 3642 6155 50  0000 L CNN
+F 2 "footprint:C_0603" H 3550 6200 50  0001 C CNN
+F 3 "" H 3550 6200 50  0000 C CNN
+	1    3550 6200
+	1    0    0    -1
+$EndComp
+$Comp
+L CP2102:CP2102 U3
+U 1 1 5893B91A
+P 2550 7100
+F 0 "U3" H 2550 7200 50  0000 C CNN
+F 1 "CP2109" H 2550 7100 50  0000 C CNN
+F 2 "Housings_DFN_QFN:QFN-28-1EP_5x5mm_Pitch0.5mm" H 2550 7100 60  0001 C CNN
+F 3 "" H 2550 7100 60  0001 C CNN
+	1    2550 7100
+	1    0    0    -1
+$EndComp
 $EndSCHEMATC
